Commit message: complete urdf visual

File: src/armbot_description/urdf/armbot.urdf.xacro (robot description, xacro)
@@ -1,5 +1,5 @@
 <?xml version="1.0"?>
 <robot xmlns:xacro="http://www.ros.org/wiki/xacro" name="armbot">
-    <xacro:property name="PI" value="3.14159"/>
+    <xacro:property name="PI" value="3.14"/>
     <xacro:property name="effort" value="30"/>
     <xacro:property name="velocity" value="10"/>
@@ -11,4 +11,7 @@
                 <mesh filename="package://armbot_description/mesh/Basement.STL" scale="0.05 0.05 0.05"/>
             </geometry>
+            <material name="orange">
+                <color rgba="${255/255} ${108/255} ${10/255} 1.0"/>
+            </material>
         </visual>
     </link>
@@ -19,6 +22,65 @@
                 <mesh filename="package://armbot_description/mesh/Base.STL" scale="0.05 0.05 0.05"/>
             </geometry>
+            <material name="orange">
+                <color rgba="${255/255} ${108/255} ${10/255} 1.0"/>
+            </material>
         </visual>
     </link>
+    <link name="vertical_arm_link">
+        <visual>
+            <origin xyz="-0.035 -0.905 2.47" rpy="0 -${PI} ${PI}"/>
+            <geometry>
+                <mesh filename="package://armbot_description/mesh/Vertical_arm.STL" scale="0.05 0.05 0.05"/>
+            </geometry>
+            <material name="orange">
+                <color rgba="${255/255} ${108/255} ${10/255} 1.0"/>
+            </material>
+        </visual>
+    </link>
+    <link name="horizontal_arm_link">
+        <visual>
+            <origin xyz="-0.022 0.2 0.01" rpy="0 -${PI} ${PI}"/>
+            <geometry>
+                <mesh filename="package://armbot_description/mesh/Horizontal_arm.STL" scale="0.05 0.05 0.05"/>
+            </geometry>
+            <material name="orange">
+                <color rgba="${255/255} ${108/255} ${10/255} 1.0"/>
+            </material>
+        </visual>
+    </link>
+    <link name="claw_support">
+        <visual>
+            <origin xyz="0.32 -0.068 -0.07" rpy="0 0 0"/>
+            <geometry>
+                <mesh filename="package://armbot_description/mesh/Claw_support.STL" scale="0.05 0.05 0.05"/>
+            </geometry>
+            <material name="orange">
+                <color rgba="${255/255} ${108/255} ${10/255} 1.0"/>
+            </material>
+        </visual>
+    </link>
+    <link name="gripper_right">
+        <visual>
+            <origin xyz="-0.03 0 0.01" rpy="0 0 0"/>
+            <geometry>
+                <mesh filename="package://armbot_description/mesh/Gripper_right.STL" scale="0.05 0.05 0.05"/>
+            </geometry>
+            <material name="orange">
+                <color rgba="${255/255} ${108/255} ${10/255} 1.0"/>
+            </material>
+        </visual>
+    </link>
+    <link name="gripper_left">
+        <visual>
+            <origin xyz="-0.03 0 0.01" rpy="${PI} 0 0"/>
+            <geometry>
+                <mesh filename="package://armbot_description/mesh/Gripper_right.STL" scale="0.05 0.05 0.05"/>
+            </geometry>
+            <material name="orange">
+                <color rgba="${255/255} ${108/255} ${10/255} 1.0"/>
+            </material>
+        </visual>
+    </link>
+    <link name="tool_link"/>
     <joint name="virtual_joint" type="fixed">
         <parent link="world"/>
@@ -33,3 +95,42 @@
         <limit lower="-${PI}" upper="${PI}" effort="${effort}" velocity="${velocity}"/>
     </joint>
+    <joint name="joint_2" type="revolute">
+        <parent link="base_link"/>
+        <child link="vertical_arm_link"/>
+        <origin xyz="0 0 0.43" rpy="0 0 0"/>
+        <axis xyz="0 1 0"/>
+        <limit lower="-${PI/2}" upper="${PI/2}" effort="${effort}" velocity="${velocity}"/>
+    </joint>
+    <joint name="joint_3" type="revolute">
+        <parent link="vertical_arm_link"/>
+        <child link="horizontal_arm_link"/>
+        <origin xyz="-0.03 0 2.52" rpy="0 0 0"/>
+        <axis xyz="0 1 0"/>
+        <limit lower="-${PI/2}" upper="${PI/2}" effort="${effort}" velocity="${velocity}"/>
+    </joint>
+    <joint name="vertical_arm_to_claw_support" type="fixed">
+        <parent link="horizontal_arm_link"/>
+        <child link="claw_support"/>
+        <origin xyz="2.11 0 0" rpy="0 0 0"/>
+    </joint>
+    <joint name="joint_4" type="revolute">
+        <parent link="claw_support"/>
+        <child link="gripper_right"/>
+        <origin xyz="0.38 -0.16 -0.03" rpy="0 0 0"/>
+        <axis xyz="0 0 1"/>
+        <limit lower="-${PI/4.7}" upper="0" effort="${effort}" velocity="${velocity}"/>
+    </joint>
+    <joint name="joint_5" type="revolute">
+        <parent link="claw_support"/>
+        <child link="gripper_left"/>
+        <origin xyz="0.38 0.02 -0.03" rpy="0 0 0"/>
+        <axis xyz="0 0 1"/>
+        <limit lower="0" upper="${PI/4.7}" effort="${effort}" velocity="${velocity}"/>
+        <mimic joint="joint_4" offset="0" multiplier="-1"/>
+    </joint>
+    <joint name="gripper_right_to_tool" type="fixed">
+        <parent link="gripper_right"/>
+        <child link="tool_link"/>
+        <origin xyz="0 0 0" rpy="0 0 0"/>
+    </joint>
 </robot>

Commit message: -add gazebo simulation -add physics properties to urdf

File: src/armbot_description/urdf/armbot.urdf.xacro (robot description, xacro)
@@ -1,9 +1,33 @@
 <?xml version="1.0"?>
 <robot xmlns:xacro="http://www.ros.org/wiki/xacro" name="armbot">
+    <!--  -->
     <xacro:property name="PI" value="3.14"/>
     <xacro:property name="effort" value="30"/>
     <xacro:property name="velocity" value="10"/>
+    <!--  -->
+    <xacro:macro name="default_inertial" params="mass">
+        <inertial>
+            <mass value="${mass}"/>
+           <inertia ixx="1" ixy="0.0" ixz="0.0" iyy="1" iyz="0.0" izz="1"/>
+        </inertial>
+    </xacro:macro>
+    <xacro:macro name="default_transmission" params="number">
+        <transmission name="transmission_${number}">
+            <type>
+                transmission_interface/SimpleTransmission
+            </type>
+            <joint name="joint_${number}">
+                <hardwareInterface>hardware_interface/PositionJointInterface</hardwareInterface>
+            </joint>
+            <actuator name="motor_${number}">
+                <hardwareInterface>hardware_interface/PositionJointInterface</hardwareInterface>
+                <mechanicalReduction>1</mechanicalReduction>
+            </actuator>
+        </transmission>
+    </xacro:macro>
+    <!--  -->
     <link name="world"/>
     <link name="basement_link">
+        <xacro:default_inertial mass="0.3"/>
         <visual>
             <origin xyz="0.0 0.0 0.0" rpy="0.0 0.0 0.0"/>
@@ -15,6 +39,13 @@
             </material>
         </visual>
+        <collision>
+            <origin xyz="0.0 0.0 0.0" rpy="0.0 0.0 0.0"/>
+            <geometry>
+                <mesh filename="package://armbot_description/mesh/Basement.STL" scale="0.05 0.05 0.05"/>
+            </geometry>
+        </collision>
     </link>
     <link name="base_link">
+        <xacro:default_inertial mass="1.0"/>
         <visual>
             <origin xyz="0.0 0.0 0.23" rpy="0.0 0.0 0.0"/>
@@ -26,6 +57,13 @@
             </material>
         </visual>
+        <collision>
+            <origin xyz="0.0 0.0 0.23" rpy="0.0 0.0 0.0"/>
+            <geometry>
+                <mesh filename="package://armbot_description/mesh/Base.STL" scale="0.05 0.05 0.05"/>
+            </geometry>
+        </collision>
     </link>
     <link name="vertical_arm_link">
+        <xacro:default_inertial mass="0.4"/>
         <visual>
             <origin xyz="-0.035 -0.905 2.47" rpy="0 -${PI} ${PI}"/>
@@ -37,6 +75,13 @@
             </material>
         </visual>
+        <collision>
+            <origin xyz="-0.035 -0.905 2.47" rpy="0 -${PI} ${PI}"/>
+            <geometry>
+                <mesh filename="package://armbot_description/mesh/Vertical_arm.STL" scale="0.05 0.05 0.05"/>
+            </geometry>
+        </collision>
     </link>
     <link name="horizontal_arm_link">
+        <xacro:default_inertial mass="0.3"/>
         <visual>
             <origin xyz="-0.022 0.2 0.01" rpy="0 -${PI} ${PI}"/>
@@ -48,6 +93,13 @@
             </material>
         </visual>
+        <collision>
+            <origin xyz="-0.022 0.2 0.01" rpy="0 -${PI} ${PI}"/>
+            <geometry>
+                <mesh filename="package://armbot_description/mesh/Horizontal_arm.STL" scale="0.05 0.05 0.05"/>
+            </geometry>
+        </collision>
     </link>
     <link name="claw_support">
+        <xacro:default_inertial mass="0.05"/>
         <visual>
             <origin xyz="0.32 -0.068 -0.07" rpy="0 0 0"/>
@@ -59,6 +111,13 @@
             </material>
         </visual>
+        <collision>
+            <origin xyz="0.32 -0.068 -0.07" rpy="0 0 0"/>
+            <geometry>
+                <mesh filename="package://armbot_description/mesh/Claw_support.STL" scale="0.05 0.05 0.05"/>
+            </geometry>
+        </collision>
     </link>
     <link name="gripper_right">
+        <xacro:default_inertial mass="0.01"/>
         <visual>
             <origin xyz="-0.03 0 0.01" rpy="0 0 0"/>
@@ -70,6 +129,13 @@
             </material>
         </visual>
+        <collision>
+            <origin xyz="-0.03 0 0.01" rpy="0 0 0"/>
+            <geometry>
+                <mesh filename="package://armbot_description/mesh/Gripper_right.STL" scale="0.05 0.05 0.05"/>
+            </geometry>
+        </collision>
     </link>
     <link name="gripper_left">
+        <xacro:default_inertial mass="0.01"/>
         <visual>
             <origin xyz="-0.03 0 0.01" rpy="${PI} 0 0"/>
@@ -81,6 +147,13 @@
             </material>
         </visual>
+        <collision>
+            <origin xyz="-0.03 0 0.01" rpy="${PI} 0 0"/>
+            <geometry>
+                <mesh filename="package://armbot_description/mesh/Gripper_right.STL" scale="0.05 0.05 0.05"/>
+            </geometry>
+        </collision>
     </link>
     <link name="tool_link"/>
+    <!--  -->
     <joint name="virtual_joint" type="fixed">
         <parent link="world"/>
@@ -134,3 +207,24 @@
         <origin xyz="0 0 0" rpy="0 0 0"/>
     </joint>
+    <!--  -->
+    <xacro:default_transmission number="1"/>
+    <xacro:default_transmission number="2"/>
+    <xacro:default_transmission number="3"/>
+    <xacro:default_transmission number="4"/>
+    <!--  -->
+    <gazebo>
+        <plugin name="gazebo_ros_control" filename="libgazebo_ros_control.so">
+            <robotNamespace>/armbot</robotNamespace>
+            <robotSimType>gazebo_ros_control/DefaultRobotHWSim</robotSimType>
+            <legacyModeNS>true</legacyModeNS>
+        </plugin>
+        <plugin name="joint_5_mimic_joint_4" filename="libroboticsgroup_gazebo_mimic_joint_plugin.so">
+            <joint>joint_4</joint>
+            <mimicJoint>joint_5</mimicJoint>
+            <multiplier>-1.0</multiplier>
+            <offset>0</offset>
+            <maxEffort>${effort}</maxEffort>
+            <robotnamespace>/armbot</robotnamespace>
+        </plugin>
+    </gazebo>
 </robot>

Commit message: fix intent for alexa

File: src/armbot_description/urdf/armbot.urdf.xacro (robot description, xacro)
@@ -139,7 +139,7 @@
         <xacro:default_inertial mass="0.01"/>
         <visual>
-            <origin xyz="-0.03 0 0.01" rpy="${PI} 0 0"/>
-            <geometry>
-                <mesh filename="package://armbot_description/mesh/Gripper_right.STL" scale="0.05 0.05 0.05"/>
+            <origin xyz="-0.03 0 0.01" rpy="0 0 0"/>
+            <geometry>
+                <mesh filename="package://armbot_description/mesh/Gripper_left.STL" scale="0.05 0.05 0.05"/>
             </geometry>
             <material name="orange">
